File: weatherstation.kicad_pcb (KiCad board)
At the start: 2 copper layers, 77.5 x 47 mm, 29 parts, among them J1 Conn_02x13_Odd_Even, J10 Conn_01x03_Male, J2 Conn_01x02_Male, J3 Conn_01x02_Male, J4 Conn_01x02_Male, J5 Conn_01x02_Male, J6 Conn_01x02_Male, J7 Conn_01x02_Male, J8 Conn_01x02_Male, J9 Conn_01x02_Male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

Commit message: Added first layout on silkscreen
Other:
- board text added: "Layout Attempt #1"
