File: weatherstation.kicad_pcb (KiCad board)
At the start: 2 copper layers, 53.3 x 53.3 mm, 30 parts, among them J1 Conn_02x13_Odd_Even, J10 Conn_01x03_Male, J2 Conn_01x02_Male, J3 Conn_01x02_Male, J4 Conn_01x02_Male, J5 Conn_01x02_Male, J6 Conn_01x02_Male, J7 Conn_01x02_Male, J8 Conn_01x02_Male, J9 Conn_01x02_Male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

Commit message: Added place for jlc order number
Parts:
- moved G*** 20.3 mm to (143.5, 115.6)
Other:
- board text added: "JLCJLCJLCJLC"
- board text added: "WindReader"
- board text removed: "eWx1"
Changed lines of the file:
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@@
   (general
     (thickness 1.6)
-    (drawings 11)
+    (drawings 12)
     (tracks 282)
     (zones 0)
@@
     (pad_to_mask_clearance 0)
     (aux_axis_origin 0 0)
+    (grid_origin 162.56 115.57)
     (visible_elements FFFFFF7F)
     (pcbplotparams
@@
   )
   (module "logodir:mylogo small" (layer F.Cu)
-    (at 163.83 115.57)
+    (at 143.51 115.57)
     (fp_text reference G*** (at 0 0) (layer F.SilkS) hide
       (effects (font (size 1.524 1.524) (thickness 0.3)))
@@
     )
   )
+  (gr_text JLCJLCJLCJLC (at 160.02 115.57) (layer B.SilkS)
+    (effects (font (size 1 1) (thickness 0.15)) (justify mirror))
+  )
   (gr_text "-\n" (at 168.91 110.49 90) (layer F.SilkS)
     (effects (font (size 1.5 1.5) (thickness 0.3)))
@@
     (effects (font (size 1 1) (thickness 0.15)))
   )
-  (gr_text eWx1 (at 154.94 115.57) (layer F.SilkS)
+  (gr_text "WindReader\n" (at 158.75 115.57) (layer F.SilkS)
     (effects (font (size 1.5 1.5) (thickness 0.3)))
   )
@@
   (segment (start 123.264998 82.55) (end 129.459999 88.745001) (width 0.25) (layer B.Cu) (net 6))
   (segment (start 119.38 82.55) (end 123.264998 82.55) (width 0.25) (layer B.Cu) (net 6))
-  (segment (start 117.21501 110.86501) (end 117.21501 84.71499) (width 0.25) (layer B.Cu) (net 6))
-  (segment (start 117.21501 84.71499) (end 119.38 82.55) (width 0.25) (layer B.Cu) (net 6))
-  (segment (start 119.38 113.03) (end 117.21501 110.86501) (width 0.25) (layer B.Cu) (net 6))
   (segment (start 119.38 115.57) (end 119.38 113.03) (width 0.25) (layer F.Cu) (net 6))
+  (segment (start 119.38 113.03) (end 117.754989 111.404989) (width 0.25) (layer B.Cu) (net 6))
+  (segment (start 117.754989 111.404989) (end 117.754989 84.175011) (width 0.25) (layer B.Cu) (net 6))
+  (segment (start 117.754989 84.175011) (end 119.38 82.55) (width 0.25) (layer B.Cu) (net 6))
   (segment (start 154.990001 66.410001) (end 157.16 68.58) (width 0.25) (layer F.Cu) (net 7))
   (segment (start 129.169999 66.410001) (end 154.990001 66.410001) (width 0.25) (layer F.Cu) (net 7))
