File: hardware/weatherstation.sch (KiCad schematic (older format))
At the start: 29 parts, among them J1 Conn_02x13_Odd_Even, J10 Conn_01x03_Male, J2 Conn_01x02_Male, J3 Conn_01x02_Male, J4 Conn_01x02_Male, J5 Conn_01x02_Male, J6 Conn_01x02_Male, J7 Conn_01x02_Male, J8 Conn_01x02_Male, J9 Conn_01x02_Male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

Commit message: Fixed ground of anemometer going ground problem
Connections:
- wire segments 100 -> 101
Changed lines of the file:
@@
 Wire Wire Line
 	1100 1200 1550 1200
-$Comp
-L power:GND #PWR0116
-U 1 1 60EDBC20
-P 1250 1400
-F 0 "#PWR0116" H 1250 1150 50  0001 C CNN
-F 1 "GND" H 1255 1227 50  0000 C CNN
-F 2 "" H 1250 1400 50  0001 C CNN
-F 3 "" H 1250 1400 50  0001 C CNN
-	1    1250 1400
-	1    0    0    -1
-$EndComp
 Wire Wire Line
 	1100 1300 1250 1300
-Wire Wire Line
-	1250 1300 1250 1400
 Text Label 5700 1450 0    50   ~ 0
 CH0
@@
 Wire Notes Line
 	650  4850 5000 4850
+Wire Wire Line
+	1250 1300 1250 1500
+Wire Wire Line
+	1250 1500 1550 1500
+Connection ~ 1550 1500
 $EndSCHEMATC
